File: FIDO2Device/MDBT50Q_Dongle/pcb_rev2_1/FIDO2AUTH_0021.brd (EAGLE design)
At the start: 19.1 x 31.8 mm, 36 parts, among them CN1 TE-1734028, CN2 IF_4PIN, SW1 SKRPACE010, SW2 SKTADAE010, U1 MDBT50Q-P1M, U2 XC6206P332MR-G, U3 ATECC608A-MAHDA-S, X1 NX3215SA-32.768K

Commit message: 配線データを作成
・ERC、DRC共にエラー無し
Parts:
- moved C3 6.11 mm to (1.27, 15.9)
- moved R1 6.05 mm to (14.3, 10.6), turned to 0 degrees
- moved C6 5.63 mm to (9.53, 14.1), turned to 180 degrees
- moved FB2 4.61 mm to (4.45, 6.03), turned to 90 degrees
- moved C8 4.43 mm to (9.53, 12.9), turned to 180 degrees
- moved R7 4.37 mm to (4.13, 26.4)
- moved C9 4.05 mm to (14.3, 11.9), turned to 180 degrees
- moved R6 3.97 mm to (8.26, 27.9)
- moved D3 3.84 mm to (4.45, 13.5), turned to 180 degrees
- moved C10 3.71 mm to (6.03, 8.26), turned to 270 degrees
- moved C11 3.41 mm to (1.59, 4.76)
- moved R8 3.35 mm to (4.13, 27.6)
- moved LED2 3.02 mm to (11.7, 30.2)
- moved C4 2.86 mm to (1.27, 12.4)
- moved LED3 2.70 mm to (8.89, 30.2)
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Connections:
- net LED2_B: now also U1.4; no longer U1.29
- net LED2_G: now also U1.6; no longer U1.26
- net LED2_R: now also U1.8; no longer U1.24
- net LED3: now also U1.10; no longer U1.20
- net SW1: now also U1.3; no longer U1.57
Routing:
- net VDD_NRF: track 0.00 -> 61.3 mm, vias 2 -> 6
- net VBUS_NRF: track 0.00 -> 26.4 mm
- net 0V: track 0.00 -> 19.7 mm, vias 4 -> 20
- net RESET: track 0.00 -> 15.4 mm
- net VBUS: track 0.00 -> 15.1 mm
- net N$3: track 0.00 -> 14.4 mm
- net TWI_SDA: track 0.00 -> 8.09 mm, vias 0 -> 2
- net SWDIO: track 0.00 -> 8.04 mm
- net TWI_SCL: track 0.00 -> 7.43 mm
- net SW1: track 0.00 -> 7.03 mm
- net N$5: track 0.00 -> 6.49 mm, vias 0 -> 1
- net N$4: track 0.00 -> 6.32 mm
- net XL1: track 0.00 -> 4.57 mm
- net SWDCLK: track 0.00 -> 4.52 mm
- net XL2: track 0.00 -> 4.52 mm
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- added copper zone on layer 1, net 0V
