File: FIDO2Device/MDBT50Q_Dongle/pcb_rev2_1/FIDO2AUTH_0021.sch (EAGLE design)
At the start: 39 parts, among them CN1 TE-1734028, CN2 IF_5PIN_H, CN3 IF_3PIN, SW1 SKRPACE010, SW2 SKTADAE010, U1 MDBT50Q-P1M, U2 XC6206P332MR-G, U3 ATECC608A-MAHDA-S, X1 NX3215SA-32.768K

Commit message: プリント基板設計データを追加
・ファイル名称を変更しています。
Parts:
- removed CN3: IF_3PIN, Connectors:IF_3PIN
- removed LED1: APHD1608LSURCK, Parts:APHD1608LSURCK
- removed R2: 1.5k, Parts:RESISTOR_0603
- C5, C7, C8, C9: device Parts:CAP_0603 -> Parts:CAP_0402
- CN2: value IF_5PIN_H -> IF_4PIN; device Connectors:IF_5PIN_H -> Connectors:IF_4PIN
- R1, R3, R4, R5, R6: device Parts:RESISTOR_0603 -> Parts:RESISTOR_0402
Connections:
- removed net AIN0: CN3.3, U1.P0.02/AIN0
- removed net LED1: R2.1, U1.P1.10
- removed net N$11: LED1.C, R2.2
- removed net UART_TX: CN3.2, U1.P0.06
- net 0V: no longer CN3.1
- net RESET: no longer CN2.5
- net SWDCLK: now also CN2.4; no longer CN2.3
- net SWDIO: now also CN2.3; no longer CN2.2
- net VDD_NRF: now also CN2.2; no longer CN2.4, LED1.A
Other:
- note added: "USBブートローダーを 書込する際に使用します。"
- note removed: "LED（赤色）"
- note removed: "nRF52840アプリケーションを 書込する際に使用します。"

Commit message: 配線データを作成
・ERC、DRC共にエラー無し
Connections:
- net LED2_B: now also U1.P1.11; no longer U1.P0.12
- net LED2_G: now also U1.P1.13; no longer U1.P1.09
- net LED2_R: now also U1.P1.15; no longer U1.P0.08
- net LED3: now also U1.P0.29/AIN5; no longer U1.P0.04/AIN2
- net SW1: now also U1.P1.10; no longer U1.P1.06
Changed lines of the file:
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@@
 <net name="LED2_R" class="0">
 <segment>
-<pinref part="U1" gate="G$1" pin="P0.08"/>
-<wire x1="73.66" y1="45.72" x2="73.66" y2="12.7" width="0.1524" layer="91"/>
-<wire x1="73.66" y1="12.7" x2="104.14" y2="12.7" width="0.1524" layer="91"/>
-<label x="104.14" y="12.7" size="1.778" layer="95" xref="yes"/>
+<pinref part="U1" gate="G$1" pin="P1.15"/>
+<wire x1="43.18" y1="93.98" x2="35.56" y2="93.98" width="0.1524" layer="91"/>
+<label x="35.56" y="93.98" size="1.778" layer="95" rot="R180" xref="yes"/>
 </segment>
 </net>
 <net name="LED2_G" class="0">
 <segment>
-<pinref part="U1" gate="G$1" pin="P1.09"/>
-<wire x1="78.74" y1="45.72" x2="78.74" y2="17.78" width="0.1524" layer="91"/>
-<wire x1="78.74" y1="17.78" x2="104.14" y2="17.78" width="0.1524" layer="91"/>
-<label x="104.14" y="17.78" size="1.778" layer="95" xref="yes"/>
+<pinref part="U1" gate="G$1" pin="P1.13"/>
+<wire x1="43.18" y1="99.06" x2="35.56" y2="99.06" width="0.1524" layer="91"/>
+<label x="35.56" y="99.06" size="1.778" layer="95" rot="R180" xref="yes"/>
 </segment>
 </net>
 <net name="LED2_B" class="0">
 <segment>
-<pinref part="U1" gate="G$1" pin="P0.12"/>
-<wire x1="86.36" y1="45.72" x2="86.36" y2="22.86" width="0.1524" layer="91"/>
-<wire x1="86.36" y1="22.86" x2="104.14" y2="22.86" width="0.1524" layer="91"/>
-<label x="104.14" y="22.86" size="1.778" layer="95" xref="yes"/>
+<pinref part="U1" gate="G$1" pin="P1.11"/>
+<wire x1="43.18" y1="104.14" x2="35.56" y2="104.14" width="0.1524" layer="91"/>
+<label x="35.56" y="104.14" size="1.778" layer="95" rot="R180" xref="yes"/>
 </segment>
 </net>
 <net name="SW1" class="0">
-<segment>
-<pinref part="U1" gate="G$1" pin="P1.06"/>
-<wire x1="43.18" y1="144.78" x2="35.56" y2="144.78" width="0.1524" layer="91"/>
-<label x="35.56" y="144.78" size="1.778" layer="95" rot="R180" xref="yes"/>
-</segment>
 <segment>
 <pinref part="SW1" gate="G$1" pin="P"/>
@@
 <junction x="185.42" y="43.18"/>
 </segment>
+<segment>
+<pinref part="U1" gate="G$1" pin="P1.10"/>
+<wire x1="43.18" y1="114.3" x2="35.56" y2="114.3" width="0.1524" layer="91"/>
+<label x="35.56" y="114.3" size="1.778" layer="95" rot="R180" xref="yes"/>
+</segment>
 </net>
 <net name="LED3" class="0">
 <segment>
-<pinref part="U1" gate="G$1" pin="P0.04/AIN2"/>
-<wire x1="63.5" y1="45.72" x2="63.5" y2="12.7" width="0.1524" layer="91"/>
-<wire x1="63.5" y1="12.7" x2="45.72" y2="12.7" width="0.1524" layer="91"/>
-<label x="45.72" y="12.7" size="1.778" layer="95" rot="R180" xref="yes"/>
+<pinref part="U1" gate="G$1" pin="P0.29/AIN5"/>
+<wire x1="43.18" y1="88.9" x2="35.56" y2="88.9" width="0.1524" layer="91"/>
+<label x="35.56" y="88.9" size="1.778" layer="95" rot="R180" xref="yes"/>
 </segment>
 </net>
