File: FIDO2Device/BT40Dongle/pcb_rev1/SECDONGL_001.sch (EAGLE design)
At the start: 38 parts, among them CN1 CX60-24S-UNIT, CN2 IF_5PIN_H, CN3 IF_2PIN_SOL, SW1 SKRPACE010, SW2 SKRPACE010, SW3 SKTADAE010, U1 BT40, U2 ADP122ACPZ-3.3-R7, U3 RV-3028-C7

Commit message: 機能修正
・SUB SWを削除
（スイッチを１点に変更。配置スペースが無いための措置）
・回路図を修正
Parts:
- removed SW2: SKRPACE010, Parts:SKRPACE010
Connections:
- removed net SW2: SW2.P, SW2.P1, U1.P0.24
- net 0V: no longer SW2.S, SW2.S1
Other:
- note removed: "SUB SW"
- moved on the sheet: SW1
Changed lines of the file:
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@@
 <part name="GND2" library="Supply" deviceset="0V" device=""/>
 <part name="GND11" library="Supply" deviceset="0V" device=""/>
-<part name="GND13" library="Supply" deviceset="0V" device=""/>
 <part name="GND12" library="Supply" deviceset="0V" device=""/>
 <part name="SW3" library="Parts" deviceset="SKTADAE010" device=""/>
 <part name="SW1" library="Parts" deviceset="SKRPACE010" device=""/>
-<part name="SW2" library="Parts" deviceset="SKRPACE010" device=""/>
 <part name="GND1" library="Supply" deviceset="0V" device=""/>
 <part name="GND4" library="Supply" deviceset="0V" device=""/>
@@
 <text x="205.74" y="147.32" size="2.54" layer="91">バイパスコンデンサー</text>
 <text x="213.36" y="81.28" size="2.54" layer="91">リセット回路</text>
-<text x="111.76" y="45.72" size="2.54" layer="91">SUB SW</text>
 <text x="20.32" y="157.48" size="3.81" layer="91">モジュール部</text>
-<text x="55.88" y="45.72" size="2.54" layer="91">MAIN SW</text>
+<text x="88.9" y="50.8" size="2.54" layer="91">MAIN SW</text>
 </plain>
 <instances>
@@
 <instance part="GND2" gate="1" x="220.98" y="101.6"/>
 <instance part="GND11" gate="1" x="231.14" y="55.88"/>
-<instance part="GND13" gate="1" x="129.54" y="20.32"/>
-<instance part="GND12" gate="1" x="73.66" y="20.32"/>
+<instance part="GND12" gate="1" x="106.68" y="25.4"/>
 <instance part="SW3" gate="G$1" x="220.98" y="66.04" rot="R270"/>
-<instance part="SW1" gate="G$1" x="63.5" y="30.48" rot="R270"/>
-<instance part="SW2" gate="G$1" x="119.38" y="30.48" rot="R270"/>
+<instance part="SW1" gate="G$1" x="96.52" y="35.56" rot="R270"/>
 <instance part="GND1" gate="1" x="20.32" y="132.08"/>
 <instance part="GND4" gate="1" x="58.42" y="86.36"/>
@@
 </segment>
 <segment>
-<pinref part="SW2" gate="G$1" pin="S1"/>
-<pinref part="GND13" gate="1" pin="0V"/>
-<wire x1="124.46" y1="27.94" x2="129.54" y2="27.94" width="0.1524" layer="91"/>
-<wire x1="129.54" y1="27.94" x2="129.54" y2="22.86" width="0.1524" layer="91"/>
-<pinref part="SW2" gate="G$1" pin="S"/>
-<wire x1="124.46" y1="30.48" x2="129.54" y2="30.48" width="0.1524" layer="91"/>
-<wire x1="129.54" y1="30.48" x2="129.54" y2="27.94" width="0.1524" layer="91"/>
-<junction x="129.54" y="27.94"/>
-</segment>
-<segment>
 <pinref part="SW1" gate="G$1" pin="S"/>
 <pinref part="GND12" gate="1" pin="0V"/>
-<wire x1="68.58" y1="30.48" x2="73.66" y2="30.48" width="0.1524" layer="91"/>
-<wire x1="73.66" y1="30.48" x2="73.66" y2="27.94" width="0.1524" layer="91"/>
+<wire x1="101.6" y1="35.56" x2="106.68" y2="35.56" width="0.1524" layer="91"/>
+<wire x1="106.68" y1="35.56" x2="106.68" y2="33.02" width="0.1524" layer="91"/>
 <pinref part="SW1" gate="G$1" pin="S1"/>
-<wire x1="73.66" y1="27.94" x2="73.66" y2="22.86" width="0.1524" layer="91"/>
-<wire x1="68.58" y1="27.94" x2="73.66" y2="27.94" width="0.1524" layer="91"/>
-<junction x="73.66" y="27.94"/>
+<wire x1="106.68" y1="33.02" x2="106.68" y2="27.94" width="0.1524" layer="91"/>
+<wire x1="101.6" y1="33.02" x2="106.68" y2="33.02" width="0.1524" layer="91"/>
+<junction x="106.68" y="33.02"/>
 </segment>
 <segment>
@@
 </segment>
 </net>
-<net name="SW2" class="0">
-<segment>
-<pinref part="SW2" gate="G$1" pin="P"/>
-<wire x1="114.3" y1="30.48" x2="109.22" y2="30.48" width="0.1524" layer="91"/>
-<pinref part="SW2" gate="G$1" pin="P1"/>
-<wire x1="114.3" y1="27.94" x2="109.22" y2="27.94" width="0.1524" layer="91"/>
-<wire x1="109.22" y1="27.94" x2="109.22" y2="30.48" width="0.1524" layer="91"/>
-<wire x1="109.22" y1="30.48" x2="104.14" y2="30.48" width="0.1524" layer="91"/>
-<junction x="109.22" y="30.48"/>
-<label x="104.14" y="30.48" size="1.778" layer="95" rot="R180" xref="yes"/>
-</segment>
-<segment>
-<pinref part="U1" gate="G$1" pin="P0.24"/>
-<wire x1="101.6" y1="93.98" x2="101.6" y2="76.2" width="0.1524" layer="91"/>
+<net name="SW1" class="0">
+<segment>
+<pinref part="SW1" gate="G$1" pin="P"/>
+<wire x1="91.44" y1="35.56" x2="86.36" y2="35.56" width="0.1524" layer="91"/>
+<pinref part="SW1" gate="G$1" pin="P1"/>
+<wire x1="86.36" y1="35.56" x2="81.28" y2="35.56" width="0.1524" layer="91"/>
+<wire x1="91.44" y1="33.02" x2="86.36" y2="33.02" width="0.1524" layer="91"/>
+<wire x1="86.36" y1="33.02" x2="86.36" y2="35.56" width="0.1524" layer="91"/>
+<junction x="86.36" y="35.56"/>
+<label x="81.28" y="35.56" size="1.778" layer="95" rot="R180" xref="yes"/>
+</segment>
+<segment>
+<pinref part="U1" gate="G$1" pin="P0.23"/>
+<wire x1="104.14" y1="93.98" x2="104.14" y2="76.2" width="0.1524" layer="91"/>
+<wire x1="104.14" y1="76.2" x2="88.9" y2="76.2" width="0.1524" layer="91"/>
 <label x="88.9" y="76.2" size="1.778" layer="95" rot="R180" xref="yes"/>
-<wire x1="88.9" y1="76.2" x2="101.6" y2="76.2" width="0.1524" layer="91"/>
-</segment>
-</net>
-<net name="SW1" class="0">
-<segment>
-<pinref part="SW1" gate="G$1" pin="P"/>
-<wire x1="58.42" y1="30.48" x2="53.34" y2="30.48" width="0.1524" layer="91"/>
-<pinref part="SW1" gate="G$1" pin="P1"/>
-<wire x1="53.34" y1="30.48" x2="48.26" y2="30.48" width="0.1524" layer="91"/>
-<wire x1="58.42" y1="27.94" x2="53.34" y2="27.94" width="0.1524" layer="91"/>
-<wire x1="53.34" y1="27.94" x2="53.34" y2="30.48" width="0.1524" layer="91"/>
-<junction x="53.34" y="30.48"/>
-<label x="48.26" y="30.48" size="1.778" layer="95" rot="R180" xref="yes"/>
-</segment>
-<segment>
-<pinref part="U1" gate="G$1" pin="P0.23"/>
-<wire x1="104.14" y1="93.98" x2="104.14" y2="71.12" width="0.1524" layer="91"/>
-<wire x1="104.14" y1="71.12" x2="88.9" y2="71.12" width="0.1524" layer="91"/>
-<label x="88.9" y="71.12" size="1.778" layer="95" rot="R180" xref="yes"/>
 </segment>
 </net>
@@
 <segment>
 <pinref part="U1" gate="G$1" pin="P0.28"/>
-<wire x1="119.38" y1="93.98" x2="119.38" y2="60.96" width="0.1524" layer="91"/>
-<wire x1="119.38" y1="60.96" x2="88.9" y2="60.96" width="0.1524" layer="91"/>
-<label x="88.9" y="60.96" size="1.778" layer="95" rot="R180" xref="yes"/>
+<wire x1="119.38" y1="93.98" x2="119.38" y2="66.04" width="0.1524" layer="91"/>
+<wire x1="119.38" y1="66.04" x2="88.9" y2="66.04" width="0.1524" layer="91"/>
+<label x="88.9" y="66.04" size="1.778" layer="95" rot="R180" xref="yes"/>
 </segment>
 </net>
@@
 <segment>
 <pinref part="U1" gate="G$1" pin="P0.20"/>
-<wire x1="106.68" y1="93.98" x2="106.68" y2="66.04" width="0.1524" layer="91"/>
-<wire x1="106.68" y1="66.04" x2="88.9" y2="66.04" width="0.1524" layer="91"/>
-<label x="88.9" y="66.04" size="1.778" layer="95" rot="R180" xref="yes"/>
-</segment>
-</net>
+<wire x1="106.68" y1="93.98" x2="106.68" y2="71.12" width="0.1524" layer="91"/>
+<wire x1="106.68" y1="71.12" x2="88.9" y2="71.12" width="0.1524" layer="91"/>
+<label x="88.9" y="71.12" size="1.778" layer="95" rot="R180" xref="yes"/>
+</segment>
+</net>

Commit message: 機能修正
・LEDをArduino互換Pinへ接続させるよう、回路図を修正
（P1.12〜P1.15を、それぞれLED1〜4に接続）
Connections:
- net LED1: now also U1.P1.12; no longer U1.P0.28
- net LED2: now also U1.P1.13; no longer U1.P0.29
- net LED3: now also U1.P1.14; no longer U1.P0.30
- net LED4: now also U1.P1.15; no longer U1.P0.31
Other:
- moved on the sheet: C1, SW1, SW3, U1

Commit message: 回路図を修正
・部品番号を修正
Parts:
- renumbered LD1 to LED1, LD2 to LED2, LD3 to LED3, LD4 to LED4, SW3 to SW2
Changed lines of the file:
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@@
 <part name="GND11" library="Supply" deviceset="0V" device=""/>
 <part name="GND12" library="Supply" deviceset="0V" device=""/>
-<part name="SW3" library="Parts" deviceset="SKTADAE010" device=""/>
+<part name="SW2" library="Parts" deviceset="SKTADAE010" device=""/>
 <part name="SW1" library="Parts" deviceset="SKRPACE010" device=""/>
 <part name="GND1" library="Supply" deviceset="0V" device=""/>
@@
 <part name="R5" library="Parts" deviceset="RESISTOR" device="_0402" value="390"/>
 <part name="GND15" library="Supply" deviceset="0V" device=""/>
-<part name="LD1" library="Parts" deviceset="APTD1608" device="LSECK/J4-PF" value="APTD1608LSECK/J4-PF"/>
+<part name="LED1" library="Parts" deviceset="APTD1608" device="LSECK/J4-PF" value="APTD1608LSECK/J4-PF"/>
 <part name="R2" library="Parts" deviceset="RESISTOR" device="_0402" value="1.2k"/>
-<part name="LD3" library="Parts" deviceset="APTD1608" device="LZGCK" value="APTD1608LZGCK"/>
-<part name="LD2" library="Parts" deviceset="APHD1608" device="LSURCK"/>
-<part name="LD4" library="Parts" deviceset="APTD1608" device="LVBC/D"/>
+<part name="LED3" library="Parts" deviceset="APTD1608" device="LZGCK" value="APTD1608LZGCK"/>
+<part name="LED2" library="Parts" deviceset="APHD1608" device="LSURCK"/>
+<part name="LED4" library="Parts" deviceset="APTD1608" device="LVBC/D"/>
 <part name="C6" library="Parts" deviceset="CAP" device="_0603" value="1uF"/>
 <part name="C7" library="Parts" deviceset="CAP" device="_0603" value="1uF"/>
@@
 <instance part="GND11" gate="1" x="139.7" y="25.4"/>
 <instance part="GND12" gate="1" x="78.74" y="25.4"/>
-<instance part="SW3" gate="G$1" x="129.54" y="35.56" rot="R270"/>
+<instance part="SW2" gate="G$1" x="129.54" y="35.56" rot="R270"/>
 <instance part="SW1" gate="G$1" x="68.58" y="35.56" rot="R270"/>
 <instance part="GND1" gate="1" x="25.4" y="129.54"/>
@@
 </segment>
 <segment>
-<pinref part="SW3" gate="G$1" pin="S1"/>
+<pinref part="SW2" gate="G$1" pin="S1"/>
 <pinref part="GND11" gate="1" pin="0V"/>
 <wire x1="134.62" y1="33.02" x2="139.7" y2="33.02" width="0.1524" layer="91"/>
 <wire x1="139.7" y1="33.02" x2="139.7" y2="27.94" width="0.1524" layer="91"/>
-<pinref part="SW3" gate="G$1" pin="S"/>
+<pinref part="SW2" gate="G$1" pin="S"/>
 <wire x1="134.62" y1="35.56" x2="139.7" y2="35.56" width="0.1524" layer="91"/>
 <wire x1="139.7" y1="35.56" x2="139.7" y2="33.02" width="0.1524" layer="91"/>
@@
 <net name="RESET" class="0">
 <segment>
-<pinref part="SW3" gate="G$1" pin="P"/>
+<pinref part="SW2" gate="G$1" pin="P"/>
 <wire x1="124.46" y1="35.56" x2="119.38" y2="35.56" width="0.1524" layer="91"/>
-<pinref part="SW3" gate="G$1" pin="P1"/>
+<pinref part="SW2" gate="G$1" pin="P1"/>
 <wire x1="119.38" y1="35.56" x2="114.3" y2="35.56" width="0.1524" layer="91"/>
 <wire x1="124.46" y1="33.02" x2="119.38" y2="33.02" width="0.1524" layer="91"/>
@@
 <instance part="R5" gate="G$1" x="139.7" y="33.02" rot="R90"/>
 <instance part="GND15" gate="1" x="215.9" y="50.8"/>
-<instance part="LD1" gate="G$1" x="33.02" y="53.34" smashed="yes">
+<instance part="LED1" gate="G$1" x="33.02" y="53.34" smashed="yes">
 <attribute name="NAME" x="36.576" y="51.308" size="1.778" layer="95"/>
 <attribute name="VALUE" x="36.195" y="48.768" size="1.778" layer="96"/>
 </instance>
 <instance part="R2" gate="G$1" x="33.02" y="33.02" rot="R90"/>
-<instance part="LD3" gate="G$1" x="104.14" y="53.34" smashed="yes">
+<instance part="LED3" gate="G$1" x="104.14" y="53.34" smashed="yes">
 <attribute name="NAME" x="107.696" y="51.308" size="1.778" layer="95"/>
 <attribute name="VALUE" x="107.315" y="48.768" size="1.778" layer="96"/>
 </instance>
-<instance part="LD2" gate="G$1" x="68.58" y="53.34" smashed="yes">
+<instance part="LED2" gate="G$1" x="68.58" y="53.34" smashed="yes">
 <attribute name="NAME" x="72.136" y="51.308" size="1.778" layer="95"/>
 <attribute name="VALUE" x="71.755" y="48.768" size="1.778" layer="96"/>
 </instance>
-<instance part="LD4" gate="G$1" x="139.7" y="53.34" smashed="yes">
+<instance part="LED4" gate="G$1" x="139.7" y="53.34" smashed="yes">
 <attribute name="NAME" x="143.256" y="51.308" size="1.778" layer="95"/>
 <attribute name="VALUE" x="142.875" y="48.768" size="1.778" layer="96"/>
@@
 <segment>
 <label x="68.58" y="60.96" size="1.778" layer="95" rot="R90" xref="yes"/>
-<pinref part="LD2" gate="G$1" pin="A"/>
+<pinref part="LED2" gate="G$1" pin="A"/>
 <wire x1="68.58" y1="55.88" x2="68.58" y2="60.96" width="0.1524" layer="91"/>
 </segment>
@@
 </segment>
 <segment>
-<pinref part="LD1" gate="G$1" pin="A"/>
+<pinref part="LED1" gate="G$1" pin="A"/>
 <wire x1="33.02" y1="55.88" x2="33.02" y2="60.96" width="0.1524" layer="91"/>
 <label x="33.02" y="60.96" size="1.778" layer="95" rot="R90" xref="yes"/>
@@
 <segment>
 <label x="104.14" y="60.96" size="1.778" layer="95" rot="R90" xref="yes"/>
-<pinref part="LD3" gate="G$1" pin="A"/>
+<pinref part="LED3" gate="G$1" pin="A"/>
 <wire x1="104.14" y1="55.88" x2="104.14" y2="60.96" width="0.1524" layer="91"/>
 </segment>
 <segment>
 <label x="139.7" y="60.96" size="1.778" layer="95" rot="R90" xref="yes"/>
-<pinref part="LD4" gate="G$1" pin="A"/>
+<pinref part="LED4" gate="G$1" pin="A"/>
 <wire x1="139.7" y1="55.88" x2="139.7" y2="60.96" width="0.1524" layer="91"/>
 </segment>
@@
 <net name="N$8" class="0">
 <segment>
-<pinref part="LD1" gate="G$1" pin="C"/>
+<pinref part="LED1" gate="G$1" pin="C"/>
 <pinref part="R2" gate="G$1" pin="2"/>
 <wire x1="33.02" y1="48.26" x2="33.02" y2="43.18" width="0.1524" layer="91"/>
@@
 <segment>
 <pinref part="R5" gate="G$1" pin="2"/>
-<pinref part="LD4" gate="G$1" pin="C"/>
+<pinref part="LED4" gate="G$1" pin="C"/>
 <wire x1="139.7" y1="43.18" x2="139.7" y2="48.26" width="0.1524" layer="91"/>
 </segment>
@@
 <segment>
 <pinref part="R4" gate="G$1" pin="2"/>
-<pinref part="LD3" gate="G$1" pin="C"/>
+<pinref part="LED3" gate="G$1" pin="C"/>
 <wire x1="104.14" y1="43.18" x2="104.14" y2="48.26" width="0.1524" layer="91"/>
 </segment>
@@
 <segment>
 <pinref part="R3" gate="G$1" pin="2"/>
-<pinref part="LD2" gate="G$1" pin="C"/>
+<pinref part="LED2" gate="G$1" pin="C"/>
 <wire x1="68.58" y1="43.18" x2="68.58" y2="48.26" width="0.1524" layer="91"/>
 </segment>

Commit message: 回路図を修正
・誤字訂正
Other:
- note added: "ボタン乾電池ケースは 基板の裏面に実装"
- note removed: "ボタン乾電池ケースは 基板の表面に実装"
Changed lines of the file:
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@@
 <setting verticaltext="up"/>
 </settings>
-<grid distance="0.1" unitdist="inch" unit="inch" style="lines" multiple="1" display="no" altdistance="0.01" altunitdist="inch" altunit="inch"/>
+<grid distance="0.1" unitdist="inch" unit="inch" style="lines" multiple="1" display="yes" altdistance="0.01" altunitdist="inch" altunit="inch"/>
 <layers>
 <layer number="1" name="Top" color="4" fill="1" visible="no" active="no"/>
@@
 <segment>
 <pinref part="U1" gate="G$1" pin="VDD_NRF"/>
-<wire x1="172.72" y1="111.76" x2="195.58" y2="111.76" width="0.1524" layer="91"/>
-<wire x1="195.58" y1="111.76" x2="195.58" y2="134.62" width="0.1524" layer="91"/>
-<label x="195.58" y="134.62" size="1.778" layer="95" rot="R90" xref="yes"/>
+<wire x1="172.72" y1="111.76" x2="190.5" y2="111.76" width="0.1524" layer="91"/>
+<wire x1="190.5" y1="111.76" x2="190.5" y2="134.62" width="0.1524" layer="91"/>
+<label x="190.5" y="134.62" size="1.778" layer="95" rot="R90" xref="yes"/>
 </segment>
 <segment>
@@
 乾電池ホルダーにボタン乾電池を装着した場合は、3.0Vを供給します。</text>
 <text x="76.2" y="78.74" size="2.54" layer="91">ボタン乾電池ケースは
-基板の表面に実装</text>
+基板の裏面に実装</text>
 <text x="175.26" y="119.38" size="3.81" layer="91">ユーティリティーI/F部</text>
 <text x="182.88" y="111.76" size="2.1844" layer="91">TXD: UARTデバッグ出力</text>
