File: FIDO2Device/BT40SlimBoard/pcb_rev1_1/SECUREBRD_002.sch (EAGLE design)
At the start: 36 parts, among them CN1 USB4105-GF-A, CN3 IF_6PIN, SW1 SKRPACE010, SW2 SKTADAE010, U1 BT40, U2 ADP122ACPZ-3.3-R7, U3 RV-3028-C7

Commit message: 回路図を修正
・CMOS降圧器 --> LDO降圧器に変更
・一部使用部品の定数を変更
Parts:
- removed C9: 0.1uF, Parts:CAP_0402K
- R4: value 1k -> 1.2k
- R9: value 390 -> 10k
- U2: value ADP122ACPZ-3.3-R7 -> XC6206P332MR-G; device ICs:ADP122ACPZ-3.3-R7 -> Parts:XC6206P332MR-G
Connections:
- removed net N$3: C6.1, D2.A, U2.VOUT
- new net N$4: C7.1, D2.A, U2.VOUT
- net 0V: now also R9.1, U2.VSS; no longer C9.2, U2.GND
- net N$9: now also R9.2; no longer C9.1, R9.1
- net VBUS_NRF: now also C6.1; no longer C7.1, U2.EN
- net VDD_BAT: no longer R9.2
Other:
- note added: "ボタン乾電池を装着すると、常時給電されます。"
- note removed: "常時給電が必要なため、ボタン乾電池に接続します。"
- moved on the sheet: BAT1, C6, C7, C8, D2, D3, R6, R7, R8, R9, U3
