File: FIDO2Device/MDBT50Q_Dongle/pcb_rev2_2/FIDO2AUTH_0022.sch (EAGLE design)
At the start: 40 parts, among them CN1 TE-1734028, CN2 IF_5PIN_H, SW1 SKRPACE010, SW2 SKTADAE010, U1 MDBT50Q-P1M, U2 XC6206P302MR-G, U4 RV-3028-C7, X1 NX3215SA-32.768K

Commit message: 回路図を作成
・チップ抵抗器のランドパターンを修正版に差し替え
Parts:
- R1, R10, R11, R2, R3, R4, R5, R6, R9: device Parts:RESISTOR_0402 -> Parts:RESISTOR_0402N
Changed lines of the file:
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@@
 <part name="D1" library="Parts" deviceset="PRTR5V0U2X" device=""/>
 <part name="CN1" library="Connectors" deviceset="TE-1734028" device=""/>
-<part name="R1" library="Parts" deviceset="RESISTOR" device="_0402" value="10k"/>
+<part name="R1" library="Parts" deviceset="RESISTOR" device="_0402N" value="10k"/>
 <part name="C9" library="Parts" deviceset="CAP" device="_0402K" value="0.1uF"/>
 <part name="GND11" library="Supply" deviceset="0V" device=""/>
@@
 <part name="SW2" library="Parts" deviceset="SKTADAE010" device=""/>
 <part name="GND12" library="Supply" deviceset="0V" device=""/>
-<part name="R3" library="Parts" deviceset="RESISTOR" device="_0402" value="1.2k"/>
-<part name="R4" library="Parts" deviceset="RESISTOR" device="_0402" value="1.5K"/>
-<part name="R5" library="Parts" deviceset="RESISTOR" device="_0402" value="390"/>
+<part name="R3" library="Parts" deviceset="RESISTOR" device="_0402N" value="1.2k"/>
+<part name="R4" library="Parts" deviceset="RESISTOR" device="_0402N" value="1.5K"/>
+<part name="R5" library="Parts" deviceset="RESISTOR" device="_0402N" value="390"/>
 <part name="GND14" library="Supply" deviceset="0V" device=""/>
 <part name="FRAME3" library="Generic" deviceset="A4L-LOC" device=""/>
@@
 <part name="GND18" library="Supply" deviceset="0V" device=""/>
 <part name="LD1" library="Parts" deviceset="APTD1608" device="LSECK/J4-PF" value="APTD1608LSECK/J4-PF"/>
-<part name="R6" library="Parts" deviceset="RESISTOR" device="_0402" value="1.2k"/>
+<part name="R6" library="Parts" deviceset="RESISTOR" device="_0402N" value="1.2k"/>
 <part name="LD3" library="Parts" deviceset="APTD1608" device="LZGCK" value="APTD1608LZGCK"/>
 <part name="LD2" library="Parts" deviceset="APHD1608" device="LSURCK"/>
@@
 <part name="U4" library="ICs" deviceset="RV-3028-C7" device=""/>
 <part name="GND21" library="Supply" deviceset="0V" device=""/>
-<part name="R2" library="Parts" deviceset="RESISTOR" device="_0402" value="10k"/>
-<part name="R9" library="Parts" deviceset="RESISTOR" device="_0402" value="10k"/>
-<part name="R10" library="Parts" deviceset="RESISTOR" device="_0402" value="10k"/>
+<part name="R2" library="Parts" deviceset="RESISTOR" device="_0402N" value="10k"/>
+<part name="R9" library="Parts" deviceset="RESISTOR" device="_0402N" value="10k"/>
+<part name="R10" library="Parts" deviceset="RESISTOR" device="_0402N" value="10k"/>
 <part name="C13" library="Parts" deviceset="CAP" device="_0402K" value="0.1uF"/>
-<part name="R11" library="Parts" deviceset="RESISTOR" device="_0402" value="10k"/>
+<part name="R11" library="Parts" deviceset="RESISTOR" device="_0402N" value="10k"/>
 <part name="CN2" library="Connectors" deviceset="IF_5PIN" device="_H"/>
 </parts>

Commit message: 回路図を作成
・チップコンデンサーのランドパターンを修正版に差し替え
Parts:
- C1, C10, C11, C2, C3, C4, C6: device Parts:CAP_0603 -> Parts:CAP_0603N
- C13, C5, C7, C8, C9: device Parts:CAP_0402K -> Parts:CAP_0402N
Changed lines of the file:
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@@
 <part name="FRAME1" library="Generic" deviceset="A4L-LOC" device=""/>
 <part name="X1" library="Parts" deviceset="NX3215SA" device="-32.768K"/>
-<part name="C1" library="Parts" deviceset="CAP" device="_0603" value="12pF"/>
-<part name="C2" library="Parts" deviceset="CAP" device="_0603" value="12pF"/>
+<part name="C1" library="Parts" deviceset="CAP" device="_0603N" value="12pF"/>
+<part name="C2" library="Parts" deviceset="CAP" device="_0603N" value="12pF"/>
 <part name="GND1" library="Supply" deviceset="0V" device=""/>
-<part name="C3" library="Parts" deviceset="CAP" device="_0603" value="4.7uF"/>
-<part name="C4" library="Parts" deviceset="CAP" device="_0603" value="4.7uF"/>
+<part name="C3" library="Parts" deviceset="CAP" device="_0603N" value="4.7uF"/>
+<part name="C4" library="Parts" deviceset="CAP" device="_0603N" value="4.7uF"/>
 <part name="GND2" library="Supply" deviceset="0V" device=""/>
 <part name="GND3" library="Supply" deviceset="0V" device=""/>
@@
 <part name="FB1" library="Parts" deviceset="BLM15AG" device="121SN1D"/>
 <part name="FB2" library="Parts" deviceset="BLM15AG" device="121SN1D"/>
-<part name="C5" library="Parts" deviceset="CAP" device="_0402K" value="0.01uF"/>
-<part name="C6" library="Parts" deviceset="CAP" device="_0603" value="10uF"/>
-<part name="C7" library="Parts" deviceset="CAP" device="_0402K" value="0.1uF"/>
-<part name="C8" library="Parts" deviceset="CAP" device="_0402K" value="0.1uF"/>
+<part name="C5" library="Parts" deviceset="CAP" device="_0402N" value="0.01uF"/>
+<part name="C6" library="Parts" deviceset="CAP" device="_0603N" value="10uF"/>
+<part name="C7" library="Parts" deviceset="CAP" device="_0402N" value="0.1uF"/>
+<part name="C8" library="Parts" deviceset="CAP" device="_0402N" value="0.1uF"/>
 <part name="GND8" library="Supply" deviceset="0V" device=""/>
 <part name="GND9" library="Supply" deviceset="0V" device=""/>
@@
 <part name="CN1" library="Connectors" deviceset="TE-1734028" device=""/>
 <part name="R1" library="Parts" deviceset="RESISTOR" device="_0402N" value="10k"/>
-<part name="C9" library="Parts" deviceset="CAP" device="_0402K" value="0.1uF"/>
+<part name="C9" library="Parts" deviceset="CAP" device="_0402N" value="0.1uF"/>
 <part name="GND11" library="Supply" deviceset="0V" device=""/>
 <part name="SW1" library="Parts" deviceset="SKRPACE010" device=""/>
@@
 <part name="FRAME3" library="Generic" deviceset="A4L-LOC" device=""/>
 <part name="U2" library="Parts" deviceset="XC6206" device="P302MR-G" value="XC6206P302MR-G"/>
-<part name="C10" library="Parts" deviceset="CAP" device="_0603" value="1uF"/>
-<part name="C11" library="Parts" deviceset="CAP" device="_0603" value="1uF"/>
+<part name="C10" library="Parts" deviceset="CAP" device="_0603N" value="1uF"/>
+<part name="C11" library="Parts" deviceset="CAP" device="_0603N" value="1uF"/>
 <part name="GND15" library="Supply" deviceset="0V" device=""/>
 <part name="GND16" library="Supply" deviceset="0V" device=""/>
@@
 <part name="R9" library="Parts" deviceset="RESISTOR" device="_0402N" value="10k"/>
 <part name="R10" library="Parts" deviceset="RESISTOR" device="_0402N" value="10k"/>
-<part name="C13" library="Parts" deviceset="CAP" device="_0402K" value="0.1uF"/>
+<part name="C13" library="Parts" deviceset="CAP" device="_0402N" value="0.1uF"/>
 <part name="R11" library="Parts" deviceset="RESISTOR" device="_0402N" value="10k"/>
 <part name="CN2" library="Connectors" deviceset="IF_5PIN" device="_H"/>
